File: hardware/begonia/begonia.sch (KiCad schematic (older format))
At the start: 13 parts, among them J1 NEIGHBOR1, J2 NEIGHBOR2, J7 BONUS_ROW, P1 POGOPINS, SW1 SPST

Commit message: daffodil: oops, J7 should not be DNP
Parts:
- J1, J2: Description (none) -> CONN RCPT .100\" 40POS DUAL-ROW STACKING GOLD; Manufacturer (none) -> Samtec; Note (none) -> Alternate: https://www.adafruit.com/products/2223; Part Number (none) -> SSQ-120-23-G-D
- J7: Description (none) -> CONN RCPT .100\" 20POS SINGLE-ROW STACKING GOLD; Manufacturer (none) -> Samtec; Part Number (none) -> SSQ-120-23-G-S
Changed lines of the file:
@@
 F 2 "gsg-modules:HEADER-2x20" H 9150 1700 60  0001 C CNN
 F 3 "" H 9150 1700 60  0000 C CNN
+F 4 "Samtec" H 9150 2650 60  0001 C CNN "Manufacturer"
+F 5 "SSQ-120-23-G-D" H 9150 2650 60  0001 C CNN "Part Number"
+F 6 "CONN RCPT .100\" 40POS DUAL-ROW STACKING GOLD" H 9150 2650 60  0001 C CNN "Description"
+F 7 "Alternate: https://www.adafruit.com/products/2223" H 9150 2650 60  0001 C CNN "Note"
 	1    9150 2650
 	1    0    0    -1
@@
 F 2 "gsg-modules:HEADER-2x20" H 9150 4300 60  0001 C CNN
 F 3 "" H 9150 4300 60  0000 C CNN
+F 4 "Samtec" H 9150 5250 60  0001 C CNN "Manufacturer"
+F 5 "SSQ-120-23-G-D" H 9150 5250 60  0001 C CNN "Part Number"
+F 6 "CONN RCPT .100\" 40POS DUAL-ROW STACKING GOLD" H 9150 5250 60  0001 C CNN "Description"
+F 7 "Alternate: https://www.adafruit.com/products/2223" H 9150 5250 60  0001 C CNN "Note"
 	1    9150 5250
 	1    0    0    -1
@@
 F 2 "gsg-modules:HEADER-1x20" H 4000 7000 60  0001 C CNN
 F 3 "" H 4000 7000 60  0000 C CNN
-F 4 "DNP" V 4250 7000 60  0000 C CNN "Note"
+F 4 "Samtec" H 4000 7000 60  0001 C CNN "Manufacturer"
+F 5 "SSQ-120-23-G-S" H 4000 7000 60  0001 C CNN "Part Number"
+F 6 "CONN RCPT .100\" 20POS SINGLE-ROW STACKING GOLD" H 4000 7000 60  0001 C CNN "Description"
+F 7 "DNP" V 4250 7000 60  0000 C CNN "Note"
 	1    4000 7000
 	0    -1   -1   0
